File: Mimosa-Anemo.sch (KiCad schematic (older format))
At the start: 0 parts

Commit message: update
Parts:
- added D?: D_Photo, symbol Device:D_Photo
- added D?: LED, symbol Device:LED
- added U? (x4): MPXV2010DP, symbol Sensor_Pressure:MPXV2010DP
- added U?: TLV493D, Package_TO_SOT_SMD:SOT-23-6, symbol Sensor_Magnetic:TLV493D
Changed lines of the file:
@@
 Comment4 ""
 $EndDescr
+$Comp
+L Sensor_Pressure:MPXV2010DP U?
+U 1 1 5F3ABB2F
+P 2250 1450
+F 0 "U?" H 1870 1496 50  0000 R CNN
+F 1 "MPXV2010DP" H 1870 1405 50  0000 R CNN
+F 2 "" H 2300 1450 50  0001 C CNN
+F 3 "https://www.nxp.com/docs/en/data-sheet/MPX2010.pdf" H 2300 1450 50  0001 C CNN
+	1    2250 1450
+	1    0    0    -1
+$EndComp
+$Comp
+L Sensor_Pressure:MPXV2010DP U?
+U 1 1 5F3AC50B
+P 2250 2950
+F 0 "U?" H 1870 2996 50  0000 R CNN
+F 1 "MPXV2010DP" H 1870 2905 50  0000 R CNN
+F 2 "" H 2300 2950 50  0001 C CNN
+F 3 "https://www.nxp.com/docs/en/data-sheet/MPX2010.pdf" H 2300 2950 50  0001 C CNN
+	1    2250 2950
+	1    0    0    -1
+$EndComp
+$Comp
+L Sensor_Pressure:MPXV2010DP U?
+U 1 1 5F3ACFA0
+P 2250 4400
+F 0 "U?" H 1870 4446 50  0000 R CNN
+F 1 "MPXV2010DP" H 1870 4355 50  0000 R CNN
+F 2 "" H 2300 4400 50  0001 C CNN
+F 3 "https://www.nxp.com/docs/en/data-sheet/MPX2010.pdf" H 2300 4400 50  0001 C CNN
+	1    2250 4400
+	1    0    0    -1
+$EndComp
+$Comp
+L Sensor_Pressure:MPXV2010DP U?
+U 1 1 5F3AD875
+P 2200 5950
+F 0 "U?" H 1820 5996 50  0000 R CNN
+F 1 "MPXV2010DP" H 1820 5905 50  0000 R CNN
+F 2 "" H 2250 5950 50  0001 C CNN
+F 3 "https://www.nxp.com/docs/en/data-sheet/MPX2010.pdf" H 2250 5950 50  0001 C CNN
+	1    2200 5950
+	1    0    0    -1
+$EndComp
+$Comp
+L Sensor_Magnetic:TLV493D U?
+U 1 1 5F482000
+P 5700 1500
+F 0 "U?" H 5980 1596 50  0000 L CNN
+F 1 "TLV493D" H 5980 1505 50  0000 L CNN
+F 2 "Package_TO_SOT_SMD:SOT-23-6" H 5650 1000 50  0001 C CNN
+F 3 "http://www.infineon.com/dgdl/Infineon-TLV493D-A1B6-DS-v01_00-EN.pdf?fileId=5546d462525dbac40152a6b85c760e80" H 5550 2000 50  0001 C CNN
+	1    5700 1500
+	1    0    0    -1
+$EndComp
+$Comp
+L Device:D_Photo D?
+U 1 1 5F484194
+P 7600 1350
+F 0 "D?" H 7550 1645 50  0000 C CNN
+F 1 "D_Photo" H 7550 1554 50  0000 C CNN
+F 2 "" H 7550 1350 50  0001 C CNN
+F 3 "~" H 7550 1350 50  0001 C CNN
+	1    7600 1350
+	1    0    0    -1
+$EndComp
+$Comp
+L Device:LED D?
+U 1 1 5F484D56
+P 8050 1350
+F 0 "D?" H 8043 1567 50  0000 C CNN
+F 1 "LED" H 8043 1476 50  0000 C CNN
+F 2 "" H 8050 1350 50  0001 C CNN
+F 3 "~" H 8050 1350 50  0001 C CNN
+	1    8050 1350
+	1    0    0    -1
+$EndComp
 $EndSCHEMATC
